File: pcb/can.kicad_sch (KiCad schematic)
At the start: 0 parts

Commit message: continued work on schematic
Changed lines of the file:
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@@
 (kicad_sch (version 20230121) (generator eeschema)
   (paper "A4")
-  (text "MCP2551T-I/SN" (at 109.22 81.28 0)
+  (text "MCP2551T-I/SN" (at 139.7 96.52 0)
     (effects (font (size 1.27 1.27)) (justify left bottom))
   )
-  (hierarchical_label "CAN_L" (shape bidirectional) (at 139.7 83.82 0) (fields_autoplaced)
+  (hierarchical_label "CAN_L" (shape bidirectional) (at 170.18 99.06 0) (fields_autoplaced)
     (effects (font (size 1.27 1.27)) (justify left))
   )
-  (hierarchical_label "CAN_RX" (shape output) (at 96.52 81.28 180) (fields_autoplaced)
+  (hierarchical_label "CAN_RX" (shape output) (at 127 96.52 180) (fields_autoplaced)
     (effects (font (size 1.27 1.27)) (justify right))
   )
-  (hierarchical_label "CAN_TX" (shape input) (at 96.52 78.74 180) (fields_autoplaced)
+  (hierarchical_label "CAN_TX" (shape input) (at 127 93.98 180) (fields_autoplaced)
     (effects (font (size 1.27 1.27)) (justify right))
   )
-  (hierarchical_label "CAN_H" (shape bidirectional) (at 139.7 81.28 0) (fields_autoplaced)
+  (hierarchical_label "CAN_H" (shape bidirectional) (at 170.18 96.52 0) (fields_autoplaced)
     (effects (font (size 1.27 1.27)) (justify left))
   )

Commit message: schematic mostly done
Parts:
- added C24: 100n, SMT:0603, symbol generic:C
- added IC5: MCP2551, symbol serial:MCP2551
- added R15: 120R, SMT:0603, symbol generic:R
Connections:
- net CAN_H: now also IC5.7 (CANH)
- net CAN_L: now also IC5.6 (CANL)
- net CAN_RX: now also IC5.4 (RXD)
- net CAN_TX: now also IC5.1 (TXD)
- new net: IC5.8 (RS), R15.2
- new net GND: C24.1, C24.2, IC5.2 (VSS), IC5.3 (VDD), R15.1
Other:
- note removed: "MCP2551T-I/SN"
- title: (none) -> CAN bus to RC servo adapter
Changed lines of the file:
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@@
 (kicad_sch (version 20230121) (generator eeschema)
   (paper "A4")
-  (text "MCP2551T-I/SN" (at 139.7 96.52 0)
-    (effects (font (size 1.27 1.27)) (justify left bottom))
-  )
-  (hierarchical_label "CAN_L" (shape bidirectional) (at 170.18 99.06 0) (fields_autoplaced)
+  (title_block
+    (title "CAN bus to RC servo adapter")
+    (date "2024-01-10")
+    (rev "0")
+    (comment 1 "CAN bus interface")
+  )
+  (junction (at 127 106.68) (diameter 0) (color 0 0 0 0)
+  )
+  (wire (pts (xy 139.7 111.76) (xy 137.16 111.76))
+    (stroke (width 0) (type default))
+  )
+  (wire (pts (xy 127 106.68) (xy 139.7 106.68))
+    (stroke (width 0) (type default))
+  )
+  (wire (pts (xy 154.94 101.6) (xy 165.1 101.6))
+    (stroke (width 0) (type default))
+  )
+  (wire (pts (xy 154.94 106.68) (xy 165.1 106.68))
+    (stroke (width 0) (type default))
+  )
+  (wire (pts (xy 154.94 111.76) (xy 157.48 111.76))
+    (stroke (width 0) (type default))
+  )
+  (wire (pts (xy 137.16 101.6) (xy 139.7 101.6))
+    (stroke (width 0) (type default))
+  )
+  (wire (pts (xy 157.48 119.38) (xy 157.48 121.92))
+    (stroke (width 0) (type default))
+  )
+  (wire (pts (xy 137.16 104.14) (xy 139.7 104.14))
+    (stroke (width 0) (type default))
+  )
+  (wire (pts (xy 127 116.84) (xy 127 121.92))
+    (stroke (width 0) (type default))
+  )
+  (wire (pts (xy 137.16 111.76) (xy 137.16 121.92))
+    (stroke (width 0) (type default))
+  )
+  (wire (pts (xy 127 104.14) (xy 127 106.68))
+    (stroke (width 0) (type default))
+  )
+  (wire (pts (xy 127 106.68) (xy 127 111.76))
+    (stroke (width 0) (type default))
+  )
+  (wire (pts (xy 157.48 111.76) (xy 157.48 114.3))
+    (stroke (width 0) (type default))
+  )
+  (hierarchical_label "CAN_L" (shape bidirectional) (at 165.1 106.68 0) (fields_autoplaced)
     (effects (font (size 1.27 1.27)) (justify left))
   )
-  (hierarchical_label "CAN_RX" (shape output) (at 127 96.52 180) (fields_autoplaced)
+  (hierarchical_label "CAN_RX" (shape output) (at 137.16 104.14 180) (fields_autoplaced)
     (effects (font (size 1.27 1.27)) (justify right))
   )
-  (hierarchical_label "CAN_TX" (shape input) (at 127 93.98 180) (fields_autoplaced)
+  (hierarchical_label "CAN_TX" (shape input) (at 137.16 101.6 180) (fields_autoplaced)
     (effects (font (size 1.27 1.27)) (justify right))
   )
-  (hierarchical_label "CAN_H" (shape bidirectional) (at 170.18 96.52 0) (fields_autoplaced)
+  (hierarchical_label "CAN_H" (shape bidirectional) (at 165.1 101.6 0) (fields_autoplaced)
     (effects (font (size 1.27 1.27)) (justify left))
   )
+  (symbol (lib_id "generic:GND") (at 137.16 121.92 0) (unit 1)
+    (in_bom yes) (on_board yes) (dnp no) (fields_autoplaced)
+    (property "Reference" "GND030" (at 140.97 120.65 0)
+      (effects (font (size 1.27 1.27)) hide)
+    )
+    (property "Value" "GND" (at 140.97 121.92 0)
+      (effects (font (size 1.27 1.27)) hide)
+    )
+    (property "Footprint" "" (at 137.16 121.92 0)
+      (effects (font (size 1.27 1.27)) hide)
+    )
+    (property "Datasheet" "" (at 137.16 121.92 0)
+      (effects (font (size 1.27 1.27)) hide)
+    )
+    (pin "~")
+    (instances
+      (project "pcb"
+        (path "/6bb3bad6-1a89-4624-b34d-6ddda7dd16d2/fdb1a2c0-3d58-431c-bfc9-dd28e6008cdb"
+          (reference "GND030") (unit 1)
+        )
+      )
+    )
+  )
+  (symbol (lib_id "generic:GND") (at 157.48 121.92 0) (unit 1)
+    (in_bom yes) (on_board yes) (dnp no) (fields_autoplaced)
+    (property "Reference" "GND029" (at 161.29 120.65 0)
+      (effects (font (size 1.27 1.27)) hide)
+    )
+    (property "Value" "GND" (at 161.29 121.92 0)
+      (effects (font (size 1.27 1.27)) hide)
+    )
+    (property "Footprint" "" (at 157.48 121.92 0)
+      (effects (font (size 1.27 1.27)) hide)
+    )
+    (property "Datasheet" "" (at 157.48 121.92 0)
+      (effects (font (size 1.27 1.27)) hide)
+    )
+    (pin "~")
+    (instances
+      (project "pcb"
+        (path "/6bb3bad6-1a89-4624-b34d-6ddda7dd16d2/fdb1a2c0-3d58-431c-bfc9-dd28e6008cdb"
+          (reference "GND029") (unit 1)
+        )
+      )
+    )
+  )
+  (symbol (lib_id "generic:R") (at 157.48 116.84 90) (unit 1)
+    (in_bom yes) (on_board yes) (dnp no)
+    (property "Reference" "R15" (at 158.75 116.84 90)
+      (effects (font (size 1.27 1.27)) (justify right top))
+    )
+    (property "Value" "120R" (at 158.75 116.84 90)
+      (effects (font (size 1.27 1.27)) (justify right bottom))
+    )
+    (property "Footprint" "SMT:0603" (at 158.115 119.38 0)
+      (effects (font (size 1.27 1.27)) hide)
+    )
+    (property "Datasheet" "" (at 157.48 116.84 0)
+      (effects (font (size 1.27 1.27)) hide)
+    )
+    (pin "1")
+    (pin "2")
+    (instances
+      (project "pcb"
+        (path "/6bb3bad6-1a89-4624-b34d-6ddda7dd16d2/fdb1a2c0-3d58-431c-bfc9-dd28e6008cdb"
+          (reference "R15") (unit 1)
+        )
+      )
+    )
+  )
+  (symbol (lib_id "generic:GND") (at 127 121.92 0) (unit 1)
+    (in_bom yes) (on_board yes) (dnp no) (fields_autoplaced)
+    (property "Reference" "GND031" (at 130.81 120.65 0)
+      (effects (font (size 1.27 1.27)) hide)
+    )
+    (property "Value" "GND" (at 130.81 121.92 0)
+      (effects (font (size 1.27 1.27)) hide)
+    )
+    (property "Footprint" "" (at 127 121.92 0)
+      (effects (font (size 1.27 1.27)) hide)
+    )
+    (property "Datasheet" "" (at 127 121.92 0)
+      (effects (font (size 1.27 1.27)) hide)
+    )
+    (pin "~")
+    (instances
+      (project "pcb"
+        (path "/6bb3bad6-1a89-4624-b34d-6ddda7dd16d2/fdb1a2c0-3d58-431c-bfc9-dd28e6008cdb"
+          (reference "GND031") (unit 1)
+        )
+      )
+    )
+  )
+  (symbol (lib_id "generic:5V") (at 127 104.14 0) (unit 1)
+    (in_bom yes) (on_board yes) (dnp no)
+    (property "Reference" "5V05" (at 130.81 102.87 0)
+      (effects (font (size 1.27 1.27)) hide)
+    )
+    (property "Value" "5V" (at 127 101.6 0)
+      (effects (font (size 1.27 1.27)) (justify bottom))
+    )
+    (property "Footprint" "" (at 127 104.14 0)
+      (effects (font (size 1.27 1.27)) hide)
+    )
+    (property "Datasheet" "" (at 127 104.14 0)
+      (effects (font (size 1.27 1.27)) hide)
+    )
+    (pin "~")
+    (instances
+      (project "pcb"
+        (path "/6bb3bad6-1a89-4624-b34d-6ddda7dd16d2/fdb1a2c0-3d58-431c-bfc9-dd28e6008cdb"
+          (reference "5V05") (unit 1)
+        )
+      )
+    )
+  )
+  (symbol (lib_id "serial:MCP2551") (at 147.32 106.68 0) (unit 1)
+    (in_bom yes) (on_board yes) (dnp no) (fields_autoplaced)
+    (property "Reference" "IC5" (at 147.32 96.52 0)
+      (effects (font (size 1.27 1.27)))
+    )
+    (property "Value" "MCP2551" (at 147.32 99.06 0)
+      (effects (font (size 1.27 1.27)))
+    )
+    (property "Footprint" "" (at 165.1 91.44 0)
+      (effects (font (size 1.27 1.27)) hide)
+    )
+    (property "Datasheet" "https://ww1.microchip.com/downloads/en/DeviceDoc/20001667G.pdf" (at 165.1 91.44 0)
+      (effects (font (size 1.27 1.27)) hide)
+    )
+    (property "MPN" "MCP2551T-I/SN" (at 165.1 91.44 0)
+      (effects (font (size 1.27 1.27)) hide)
+    )
+    (property "Manufacturer" "Microchip" (at 165.1 91.44 0)
+      (effects (font (size 1.27 1.27)) hide)
+    )
+    (property "DigiKey" "MCP2551T-I/SNCT-ND" (at 165.1 91.44 0)
+      (effects (font (size 1.27 1.27)) hide)
+    )
+    (pin "1")
+    (pin "2")
+    (pin "3")
+    (pin "4")
+    (pin "5")
+    (pin "6")
+    (pin "7")
+    (pin "8")
+    (instances
+      (project "pcb"
+        (path "/6bb3bad6-1a89-4624-b34d-6ddda7dd16d2/fdb1a2c0-3d58-431c-bfc9-dd28e6008cdb"
+          (reference "IC5") (unit 1)
+        )
+      )
+    )
+  )
+  (symbol (lib_id "generic:C") (at 127 114.3 0) (unit 1)
+    (in_bom yes) (on_board yes) (dnp no)
+    (property "Reference" "C24" (at 128.27 114.3 0)
+      (effects (font (size 1.27 1.27)) (justify left bottom))
+    )
+    (property "Value" "100n" (at 128.27 114.3 0)
+      (effects (font (size 1.27 1.27)) (justify left top))
+    )
+    (property "Footprint" "SMT:0603" (at 127 116.84 0)
+      (effects (font (size 1.27 1.27)) hide)
+    )
+    (property "Datasheet" "" (at 127 114.3 0)
+      (effects (font (size 1.27 1.27)) hide)
+    )
+    (pin "1")
+    (pin "2")
+    (instances
+      (project "pcb"
+        (path "/6bb3bad6-1a89-4624-b34d-6ddda7dd16d2/fdb1a2c0-3d58-431c-bfc9-dd28e6008cdb"
+          (reference "C24") (unit 1)
+        )
+      )
+    )
+  )
 )

Commit message: fixed 5V being GND net
Connections:
- net GND: no longer C24.1, IC5.3 (VDD)
- new net 5V: C24.1, IC5.3 (VDD)

Commit message: added DIP switches, footprints
Parts:
- IC5: footprint (none) -> SOP:SO-8
Changed lines of the file:
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@@
       (effects (font (size 1.27 1.27)))
     )
-    (property "Footprint" "" (at 165.1 91.44 0)
+    (property "Footprint" "SOP:SO-8" (at 165.1 91.44 0)
       (effects (font (size 1.27 1.27)) hide)
     )
