File: pcb/pcb.kicad_pcb (KiCad board)
At the start: 2 copper layers, 55 x 52.5 mm, 76 parts, among them CN1 1x4, CN10 1x2, CN11 1x2, CN2 1x8, CN3 1x8, CN4 1x8, CN5 1x4, CN6 1x2, CN7 1x2, CN9 2x5, IC1 AP2112K-3.3TRG1, IC2 STM32f103C8T, IC3 INA199B2, IC4 AP62300TWU-7, IC5 MCP2551, SW1 switch_3x4, SW2 switch_3x4, SW3 219-3LPST, X1 H130B-8.000-18-3030-EXT-TR

Commit message: worked on layout
Parts:
- removed R3: 10k, SMT:0603
- moved CN7 41.3 mm to (133.5, 82.8), turned to -90 degrees
- moved CN4 31.0 mm to (123.3, 80.3), turned to -90 degrees
- moved CN3 27.5 mm to (123.3, 82.8), turned to -90 degrees
- moved CN2 24.0 mm to (123.3, 85.4), turned to -90 degrees
- moved TP6 23.4 mm to (123.3, 108.2)
- moved TP7 22.7 mm to (125.9, 110.8)
- moved SW2 21.9 mm to (135.0, 96.0), turned to -90 degrees
- moved TP10 20.9 mm to (130.9, 110.8)
- moved CN9 20.5 mm to (125.9, 113.3), turned to -90 degrees
- moved TP9 20.3 mm to (128.4, 110.8)
- moved TP8 19.3 mm to (125.9, 108.2)
- moved SW1 19.1 mm to (109.0, 64.0)
- moved C16 18.4 mm to (124.0, 92.8), turned to 90 degrees
- moved TP2 18.0 mm to (128.4, 108.2)
- moved R4 17.0 mm to (108.5, 83.0), turned to -90 degrees
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Routing:
- net /MCU/status: track 0.00 -> 28.9 mm, vias 0 -> 2
- net /MCU/I_bat: track 0.00 -> 26.7 mm, vias 0 -> 2
- net /MCU/CH1: track 0.00 -> 26.7 mm, vias 0 -> 1
- net /MCU/CH8: track 0.00 -> 26.3 mm
- net /CAN_H: track 0.00 -> 25.7 mm
- net /MCU/ADDR1: track 0.00 -> 25.6 mm, vias 0 -> 2
- net /MCU/CH7: track 0.00 -> 24.7 mm
- net /MCU/CH2: track 0.00 -> 24.6 mm, vias 0 -> 1
- net /MCU/ADDR2: track 0.00 -> 23.3 mm, vias 0 -> 2
- net /MCU/CH6: track 0.00 -> 23.0 mm
- net /CAN_L: track 0.00 -> 21.5 mm
- net /MCU/ADDR3: track 0.00 -> 21.4 mm, vias 0 -> 2
- net /MCU/CH5: track 0.00 -> 21.3 mm
- net GND: track 0.00 -> 18.4 mm, vias 0 -> 5
- net /MCU/CH4: track 0.00 -> 18.3 mm
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- added copper zone on B.Cu, net /Battery
- added copper zone on In2.Cu, net 3V3
- added copper zone on In2.Cu, net 5V
- added copper zone on In1.Cu, net GND
Other:
- board size 55 x 52.5 mm -> 52.5 x 52.5 mm
- copper layers 2 -> 4
- board text added: "+5V"
- board text added: "1"
- board text added: "2"
- board text added: "3"
- board text added: "4"
- board text added: "5"
- board text added: "6"
- board text added: "7"
- board text added: "8"

Commit message: worked on layout
Parts:
- moved SW1 36.8 mm to (135.0, 90.0), turned to -90 degrees
- moved C2 1.70 mm to (126.5, 118.8)
- moved C4 1.46 mm to (134.2, 125.4)
- moved C6 1.46 mm to (134.2, 126.4)
- moved C1 1.04 mm to (133.5, 120.8)
- moved R11 1.00 mm to (119.6, 118.6), turned to 180 degrees
- moved C22 0.72 mm to (119.6, 119.8), turned to 180 degrees
- moved SW2 0.50 mm to (135.0, 96.5)
- moved C16 0.35 mm to (124.0, 92.4)
- moved C17 0.25 mm to (131.5, 93.0)
Routing:
- net /MCU/NRST: track 13.8 -> 40.9 mm, vias 0 -> 1
- net 5V: track 2.77 -> 12.6 mm, vias 1 -> 11
- net Net-(IC2-PA12): track 0.00 -> 7.52 mm, vias 0 -> 1
- net Net-(IC4-EN): track 0.00 -> 7.39 mm
- net 3V3: track 8.56 -> 15.4 mm, vias 3 -> 11
- net Net-(IC3-REF): track 0.00 -> 4.11 mm
- net Net-(IC4-FB): track 0.00 -> 4.10 mm
- net Net-(R10-Pad1): track 0.00 -> 2.79 mm
- net Net-(IC5-RS): track 0.00 -> 2.54 mm
- net /MCU/I_bat: track 26.7 -> 29.0 mm
- net /MCU/status: track 28.9 -> 30.5 mm
- net Net-(IC2-PB13): track 4.99 -> 6.53 mm
- net Net-(IC2-PA10): track 2.02 -> 3.55 mm
- net GND: track 18.4 -> 17.4 mm, vias 5 -> 13
- net /MCU/V_bat: track 17.9 -> 18.8 mm
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- added copper zone on F.Cu, net /Battery
- added copper zone on F.Cu, net /power supply/+
- added copper zone on F.Cu, net 3V3
- added copper zone on F.Cu, net 5V
- added copper zone on B.Cu, net GND
- added copper zone on F.Cu, net GND
- added copper zone on B.Cu, net Net-(CN6-Pad1)

Commit message: worked on pinout
Parts:
- added R3: 10k, SMT:0603, F.Cu at (155.2, 95.0)
- moved REF** 9.64 mm to (153.0, 76.0)
Changed lines of the file:
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@@
+  )
+  (footprint "SMT:0603" (layer "F.Cu")
+    (at 155.2 95)
+    (property "Field2" "")
+    (property "Sheetfile" "mcu.kicad_sch")
+    (property "Sheetname" "MCU")
+    (property "Sim.Device" "R")
+    (property "Sim.Pins" "1=+ 2=-")
+    (attr through_hole)
+    (fp_text reference "R3" (at 0 1.5) (layer "F.SilkS") hide
+        (effects (font (size 1 1) (thickness 0.15)))
+    )
+    (fp_text value "10k" (at 0 -1.5) (layer "F.Fab") hide
+        (effects (font (size 1 1) (thickness 0.15)))
+    )
+    (fp_line (start -0.8 -0.4) (end 0.8 -0.4)
+      (stroke (width 0.2) (type solid)) (layer "F.Fab"))
+    (fp_line (start -0.8 0.4) (end -0.8 -0.4)
+      (stroke (width 0.2) (type solid)) (layer "F.Fab"))
+    (fp_line (start -0.8 0.4) (end 0.8 0.4)
+      (stroke (width 0.2) (type solid)) (layer "F.Fab"))
+    (fp_line (start 0.8 0.4) (end 0.8 -0.4)
+      (stroke (width 0.2) (type solid)) (layer "F.Fab"))
+    (pad "1" smd roundrect (at -0.8 0) (size 0.97 0.8) (layers "F.Cu" "F.Paste" "F.Mask") (roundrect_rratio 0.25)
+      (net 9 "/MCU/NRST") (pintype "bidirectional"))
+    (pad "2" smd roundrect (at 0.8 0) (size 0.97 0.8) (layers "F.Cu" "F.Paste" "F.Mask") (roundrect_rratio 0.25)
+      (net 2 "3V3") (pintype "bidirectional"))
+    (model "passive.wrl"
+      (offset (xyz 0 0 0))
+      (scale (xyz 1.6 0.8 0.45))
+      (rotate (xyz 0 0 0))
+    )
   )
   (footprint "SMT:0603" (layer "F.Cu")
@@
   )
   (footprint "PCB:M3" (layer "F.Cu")
-    (at 146.179999 82.82)
+    (at 153 76)
     (attr through_hole)
     (fp_text reference "REF**" (at 0 0.5) (layer "F.SilkS") hide
@@
     (polygon
       (pts
-        (xy 112.4 116)
-        (xy 112.4 105.6)
-        (xy 119.8 105.6)
-        (xy 119.8 111.3)
-        (xy 117.2 113.9)
-        (xy 117.2 116)
+        (xy 111.4 114.5)
+        (xy 111.4 105.1)
+        (xy 120.3 105.1)
+        (xy 120.3 111.5)
+        (xy 117.2 114.4)
+        (xy 117.2 114.5)
       )
     )

Commit message: worked on layout
Parts:
- removed REF** (x4): M3, PCB:M3
- removed SW1, SW2: switch_3x4, buttons:sw_3x4
- removed TP10, TP6, TP7, TP8, TP9: test_point, PCB:test_point
- removed the TP2 at (128.4, 108.2)
- removed the TP3 at (120.8, 105.7)
- removed the TP4 at (130.9, 108.2)
- removed X1: H130B-8.000-18-3030-EXT-TR, xtal:5x3.2
- added C18: 100n, SMT:0603, F.Cu at (162.1, 112.7)
- added C19: 100n, SMT:0603, F.Cu at (162.1, 115.2)
- added C26: 100n, SMT:0603, F.Cu at (162.1, 117.7)
- added C27: 100n, SMT:0603, F.Cu at (162.1, 120.3)
- added C28: 100n, SMT:0603, F.Cu at (162.1, 122.8)
- added C29: 100n, SMT:0603, F.Cu at (162.0, 86.4)
- added C30: 100n, SMT:0603, F.Cu at (162.0, 88.4)
- added C31: 100n, SMT:0603, F.Cu at (162.0, 90.4)
- added C32: 100n, SMT:0603, F.Cu at (162.0, 92.4)
- added C33: 100n, SMT:0603, F.Cu at (162.0, 94.4)
- added C34: 100n, SMT:0603, F.Cu at (162.0, 96.4)
- added C35: 100n, SMT:0603, F.Cu at (162.0, 98.4)
- added C36: 100n, SMT:0603, F.Cu at (162.0, 100.4)
- added C9: 100n, SMT:0603, F.Cu at (162.1, 105.0)
- added CN12: 1x8, pin_headers:1x8, F.Cu at (172.8, 112.0)
- added CN8: 1x8, pin_headers:1x8, F.Cu at (170.3, 112.0)
- added D2: LED, SMT:0603, F.Cu at (184.3, 86.4)
- added IC10: SN74LVC1G17, sc70:SC70-5L, F.Cu at (166.5, 114.6)
- added IC11: SN74LVC1G17, sc70:SC70-5L, F.Cu at (166.5, 117.1)
- added IC12: SN74LVC1G17, sc70:SC70-5L, F.Cu at (166.5, 119.7)
- added IC13: SN74LVC1G17, sc70:SC70-5L, F.Cu at (166.5, 122.2)
- added IC14: SN74LVC1G17, sc70:SC70-5L, F.Cu at (165.5, 87.5)
- added IC15: SN74LVC1G17, sc70:SC70-5L, F.Cu at (168.8, 87.5)
- added IC16: SN74LVC1G17, sc70:SC70-5L, F.Cu at (172.2, 87.5)
- added IC17: SN74LVC1G17, sc70:SC70-5L, F.Cu at (175.5, 87.5)
- added IC18: SN74LVC1G17, sc70:SC70-5L, F.Cu at (178.9, 87.5)
- added IC19: SN74LVC1G17, sc70:SC70-5L, F.Cu at (165.5, 91.6)
- added IC20: SN74LVC1G17, sc70:SC70-5L, F.Cu at (168.8, 91.6)
- added IC21: SN74LVC1G17, sc70:SC70-5L, F.Cu at (172.2, 91.6)
- added IC22: NPS4053, SOT:SOT-23-6, F.Cu at (188.5, 87.5)
- added IC6: SN74LVC1G17, sc70:SC70-5L, F.Cu at (166.5, 104.4)
- added IC7: SN74LVC1G17, sc70:SC70-5L, F.Cu at (166.5, 107.0)
- added IC8: SN74LVC1G17, sc70:SC70-5L, F.Cu at (166.5, 109.5)
- added IC9: SN74LVC1G17, sc70:SC70-5L, F.Cu at (166.5, 112.0)
- added R12: 10K, SMT:0603, F.Cu at (188.1, 104.4)
- added R13: 10k, SMT:0603, F.Cu at (162.1, 103.8)
- added R18: 10k, SMT:0603, F.Cu at (162.1, 106.3)
- added R19: 10k, SMT:0603, F.Cu at (162.1, 108.9)
- added R20: 10k, SMT:0603, F.Cu at (162.1, 111.4)
- added R21: 10k, SMT:0603, F.Cu at (162.1, 113.9)
- added R22: 10k, SMT:0603, F.Cu at (162.1, 116.5)
- added R23: 10k, SMT:0603, F.Cu at (162.1, 119.0)
- added R24: 10k, SMT:0603, F.Cu at (162.1, 121.6)
- added R25: R, SMT:0603, F.Cu at (188.1, 106.4)
- added R26: R, SMT:0603, F.Cu at (184.3, 88.4)
- added R27: R, SMT:0603, F.Cu at (184.3, 90.4)
- C16, C17: value 22p -> 100n
- TP1, TP5: moved to F.Cu
- moved TP1 67.1 mm to (187.6, 108.6), turned to 0 degrees
- moved TP5 54.0 mm to (183.8, 94.6), turned to 0 degrees
- moved C16 41.0 mm to (162.1, 107.6), turned to 0 degrees
- moved C17 35.0 mm to (162.1, 110.1), turned to 0 degrees
- renumbered TP13 to TP2, TP12 to TP3, TP14 to TP4
Connections:
- C16 pad 1: Net-(IC2-OSC_OUT) -> GND
- C16 pad 2: GND -> 3V3
- C17 pad 1: Net-(IC2-OSC_IN) -> GND
- C17 pad 2: GND -> 3V3
- CN2 pad 1: /MCU/CH1 -> /OUT1
- CN2 pad 2: /MCU/CH2 -> /OUT2
- CN2 pad 3: /MCU/CH3 -> /OUT3
- CN2 pad 4: /MCU/CH4 -> /OUT4
- CN2 pad 5: /MCU/CH5 -> /OUT5
- CN2 pad 6: /MCU/CH6 -> /OUT6
- CN2 pad 7: /MCU/CH7 -> /OUT7
- CN2 pad 8: /MCU/CH8 -> /OUT8
- CN7 pad 1: 5V -> /MCU/SERVO_ENABLE
- CN7 pad 2: /Servo VCC -> /servo power supply/EN
- IC2 pad 14: Net-(IC2-PA4) -> /Input  buffers/IN_1
- IC2 pad 20: Net-(IC2-PB2) -> /Input  buffers/IN_5
- IC2 pad 26: Net-(IC2-PB13) -> /Input  buffers/IN_8
- IC2 pad 27: Net-(IC2-PB14) -> /MCU/SERVO_ENABLE
- IC2 pad 31: Net-(IC2-PA10) -> /Input  buffers/IN_2
- IC2 pad 32: Net-(IC2-PA11) -> /Input  buffers/IN_3
- IC2 pad 33: Net-(IC2-PA12) -> /Input  buffers/IN_4
- IC2 pad 40: Net-(IC2-PB4) -> /Input  buffers/IN_6
- IC2 pad 41: Net-(IC2-PB5) -> /Input  buffers/IN_7
- IC2 pad 5: Net-(IC2-OSC_IN) -> unconnected-(IC2-OSC_IN-Pad5)
- IC2 pad 6: Net-(IC2-OSC_OUT) -> unconnected-(IC2-OSC_OUT-Pad6)
- TP1 pad 1: Net-(IC2-PA4) -> /MCU/DFU
- TP5 pad 1: Net-(IC2-PB5) -> Net-(IC2-PB15)
Routing:
- net unconnected-(IC2-OSC_IN-Pad5): track 0.00 -> 12.0 mm
- net Net-(IC2-OSC_IN): track 12.0 -> 0.00 mm
- net unconnected-(IC2-OSC_OUT-Pad6): track 0.00 -> 10.1 mm
- net Net-(IC2-OSC_OUT): track 10.1 -> 0.00 mm
- net Net-(IC2-PA12): track 7.52 -> 0.00 mm, vias 1 -> 0
- net /Input  buffers/IN_4: track 0.00 -> 7.52 mm, vias 0 -> 1
- net Net-(IC2-PB13): track 6.53 -> 0.00 mm, vias 1 -> 0
- net /Input  buffers/IN_8: track 0.00 -> 6.53 mm, vias 0 -> 1
- net Net-(IC2-PB4): track 3.68 -> 0.00 mm, vias 1 -> 0
- net /Input  buffers/IN_6: track 0.00 -> 3.68 mm, vias 0 -> 1
- net Net-(IC2-PA10): track 3.55 -> 0.00 mm, vias 1 -> 0
- net /Input  buffers/IN_2: track 0.00 -> 3.55 mm, vias 0 -> 1
- net Net-(IC2-PB5): track 3.00 -> 0.00 mm, vias 1 -> 0
- net /Input  buffers/IN_7: track 0.00 -> 3.00 mm, vias 0 -> 1
- net Net-(IC2-PA11): track 2.97 -> 0.00 mm, vias 1 -> 0
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